Commit message: Up date project

File: install/my_robot_description/share/my_robot_description/urdf/common_properties.xacro (robot description, xacro)
@@ -7,10 +7,10 @@
         <color rgba="1 0 0 1" />
     </material>
-    <xacro:macro name="box__collition_inertia" params="m x y z o_xyz o_rpy">
+    <xacro:macro name="box_collition_inertia" params="m x y z o_xyz o_rpy">
         <collision>
             <geometry>
                 <box size="${x} ${y} ${z}" />
             </geometry>
-            <origin xyz="0 0 ${z/2.0}" rpy="0 0 0" />
+            <origin xyz="0 0 ${z / 2.0}" rpy="0 0 0" />
         </collision>
         <inertial>
@@ -24,9 +24,9 @@
     <xacro:macro name="cylinder_collition_inertia" params="m r l o_xyz o_rpy">
         <collision>
-            <geometry>
-                <sphere radius="${r}" />
-            </geometry>
-            <origin xyz="0.0 0.0 0.0" rpy= "0 0 0" />
-        </collision>
+                <geometry>
+                    <sphere radius="${r}" />
+                </geometry>
+                <origin xyz="0 0 0" rpy="0 0 0" />
+            </collision>
         <inertial>
             <mass value="${m}"/>
@@ -40,7 +40,7 @@
         <collision>
             <geometry>
-                <sphere radius="${r}" />
+                <sphere radius="${wheel_radius / 2.0}" />
             </geometry>
-            <origin xyz="0 0 0" rpy= "0 0 0" />
+            <origin xyz="0 0 0" rpy="0 0 0" />
         </collision>
         <inertial>

File: install/my_robot_description/share/my_robot_description/urdf/mobile_base.xacro (robot description, xacro)
@@ -1,10 +1,21 @@
 <?xml version="1.0"?>
-<robot xmlns:xacro="http://www.ros.org/wiki/xacro" >
-    <xacro:property name="base_length" value="0.6"/>
-    <xacro:property name="base_width" value="0.4"/>
-    <xacro:property name="base_height" value="0.2"/>
-    <xacro:property name="wheel_radius" value="0.1"/>
-    <xacro:property name="wheel_length" value="0.05"/>
-    <xacro:property name="wheel_caster_radius" value="0.05"/>
+<robot xmlns:xacro="http://www.ros.org/wiki/xacro">
+    <xacro:property name="base_length" value="0.6" />
+    <xacro:property name="base_width" value="0.4" />
+    <xacro:property name="base_height" value="0.2" />
+    <xacro:property name="wheel_radius" value="0.1" />
+    <xacro:property name="wheel_length" value="0.05" />
+    <link name="base_footprint" />
+    <link name="base_link">
+        <visual>
+            <geometry>
+                <box size="${base_length} ${base_width} ${base_height}" />
+            </geometry>
+            <origin xyz="0 0 ${base_height / 2.0}" rpy="0 0 0" />
+            <material name="red" />
+        </visual>
+        <xacro:box_collition_inertia m="5.0" x="${base_length}" y="${base_width}" z="${base_height}"
+                           o_xyz="0 0 ${base_height / 2.0}" o_rpy="0 0 0" />
+    </link>
     <xacro:macro name="wheel_link" params="prefix">
         <link name="${prefix}_wheel_link">
@@ -13,58 +24,45 @@
                     <cylinder radius="${wheel_radius}" length="${wheel_length}" />
                 </geometry>
-                <origin xyz="0 0 0.0" rpy= "${pi/2.0} 0 0" />
-                <material name="red" />
+                <origin xyz="0 0 0" rpy="${pi / 2.0} 0 0" />
+                <material name="purple" />
             </visual>
             <xacro:cylinder_collition_inertia m="1.0" r="${wheel_radius}" l="${wheel_length}"
-                            o_xyz="0 0 0" o_rpy="${pi/2.0} 0 0" />
+                                    o_xyz="0 0 0" o_rpy="${pi / 2.0} 0 0" />
         </link>
     </xacro:macro>
     <xacro:wheel_link prefix="right" />
     <xacro:wheel_link prefix="left" />
-    <link name="base_link">
+    <link name="caster_wheel_link">
         <visual>
             <geometry>
-                <box size="${base_length} ${base_width} ${base_height}" />
+                <sphere radius="${wheel_radius / 2.0}" />
             </geometry>
-            <origin xyz="0 0 ${base_height/2.0}" rpy="0 0 0" />
+            <origin xyz="0 0 0" rpy="0 0 0" />
             <material name="purple" />
         </visual>
-        <xacro:box__collition_inertia m="5.0" x="${base_length}" y="${base_width}" z="${base_height}"
-                            o_xyz="0 0 ${base_height/2.0}" o_rpy="0 0 0" />
+        <xacro:sphere_collition_inertia m="0.5" r="${wheel_radius / 2.0}"
+                              o_xyz="0 0 0" o_rpy="0 0 0" />
     </link>
-    <link name="base_caster_wheel_link">
-        <visual>
-            <geometry>
-                <sphere radius="${wheel_caster_radius}" />
-            </geometry>
-            <origin xyz="0 0 0" rpy= "0 0 0" />
-            <material name="red" />
-        </visual>
-        <xacro:sphere_collition_inertia m="1.0" r="${wheel_caster_radius}"
-                            o_xyz="0 0 0" o_rpy="0 0 0" />
-    </link>
-    <link name="base_foodprint" />
-    <joint name="base_foodprint_joint" type="fixed">
-        <parent link="base_foodprint"/>
-        <child link="base_link"/>
+    <joint name="base_joint" type="fixed">
+        <parent link="base_footprint" />
+        <child link="base_link" />
         <origin xyz="0 0 ${wheel_radius}" rpy="0 0 0"/>
     </joint>
-    <joint name="base_rigth_wheel_joint" type="continuous">
-        <parent link="base_link"/>
-        <child link="right_wheel_link"/>
-        <origin xyz="${- base_length/4.0} ${-(base_width+wheel_length)/2.0} 0" rpy="0 0 0"/>
-        <axis xyz="0 1 0"/>
+    <joint name="base_right_wheel_joint" type="continuous">
+        <parent link="base_link" />
+        <child link="right_wheel_link" />
+        <origin xyz="${-base_length / 4.0} ${-(base_width + wheel_length) / 2.0} 0" rpy="0 0 0" />
+        <axis xyz="0 1 0" />
     </joint>
     <joint name="base_left_wheel_joint" type="continuous">
-        <parent link="base_link"/>
-        <child link="left_wheel_link"/>
-        <origin xyz="${- base_length/4.0} ${(base_width+wheel_length)/2.0} 0" rpy="0 0 0"/>
-        <axis xyz="0 1 0"/>
+        <parent link="base_link" />
+        <child link="left_wheel_link" />
+        <origin xyz="${-base_length / 4.0} ${(base_width + wheel_length) / 2.0} 0" rpy="0 0 0" />
+        <axis xyz="0 1 0" />
     </joint>
     <joint name="base_caster_wheel_joint" type="fixed">
-        <parent link="base_link"/>
-        <child link="base_caster_wheel_link"/>
-        <origin xyz="${base_length/3.0} 0 ${-wheel_radius/2.0}" rpy="0 0 0"/>
-        <axis xyz="0 0 0"/>
+        <parent link="base_link" />
+        <child link="caster_wheel_link" />
+        <origin xyz="${base_length / 3.0} 0 ${-wheel_radius / 2.0}" rpy="0 0 0" />
     </joint>
 </robot>

File: install/my_robot_description/share/my_robot_description/urdf/mobile_base_gz.xacro (robot description, xacro)
@@ -10,9 +10,9 @@
             name="gz::sim::systems::DiffDrive">
             <left_joint>base_left_wheel_joint</left_joint>
-            <right_joint>base_rigth_wheel_joint</right_joint>
-            <wheel_sepation>0.45</wheel_sepation>
+            <right_joint>base_right_wheel_joint</right_joint>
+            <wheel_separation>0.45</wheel_separation>
             <wheel_radius>0.1</wheel_radius>
             <frame_id>odom</frame_id>
-            <child_frame_id>base_foodprint</child_frame_id>
+            <child_frame_id>base_footprint</child_frame_id>
         </plugin>
     </gazebo>
@@ -22,5 +22,5 @@
             name="gz::sim::systems::JointStatePublisher">
             <joint_name>base_left_wheel_joint</joint_name>
-            <joint_name>base_rigth_wheel_joint</joint_name>
+            <joint_name>base_right_wheel_joint</joint_name>
         </plugin>
     </gazebo>

File: install/my_robot_description/share/my_robot_description/urdf/my_robot.urdf.xacro (robot description, xacro)
@@ -3,4 +3,5 @@
     <xacro:include filename="common_properties.xacro" />
     <xacro:include filename="mobile_base.xacro"/>
+    <!-- <xacro:include filename="mobile_base_Vinc.xacro"/> -->
     <xacro:include filename="mobile_base_gz.xacro"/>
 </robot>

Commit message: Final project second course of ROS2

File: install/my_robot_description/share/my_robot_description/urdf/common_properties.xacro (robot description, xacro)
@@ -1,54 +1 @@
-<?xml version="1.0"?>
-<robot xmlns:xacro="http://www.ros.org/wiki/xacro" >
-    <material name="purple">
-        <color rgba="0.5 0 0.5 1" />
-    </material>
-    <material name="red">
-        <color rgba="1 0 0 1" />
-    </material>
-    <xacro:macro name="box_collition_inertia" params="m x y z o_xyz o_rpy">
-        <collision>
-            <geometry>
-                <box size="${x} ${y} ${z}" />
-            </geometry>
-            <origin xyz="0 0 ${z / 2.0}" rpy="0 0 0" />
-        </collision>
-        <inertial>
-            <mass value="${m}"/>
-            <origin xyz="${o_xyz}" rpy="${o_rpy}"/>
-            <inertia    ixx="${(m/12) * (y*y + z*z)}"   ixy="0"   ixz="0"
-                        iyy="${(m/12) * (x*x + z*z)}"   iyz="0"
-                        izz="${(m/12) * (x*x + y*y)}"   />
-        </inertial>
-    </xacro:macro>
-    <xacro:macro name="cylinder_collition_inertia" params="m r l o_xyz o_rpy">
-        <collision>
-                <geometry>
-                    <sphere radius="${r}" />
-                </geometry>
-                <origin xyz="0 0 0" rpy="0 0 0" />
-            </collision>
-        <inertial>
-            <mass value="${m}"/>
-            <origin xyz="${o_xyz}" rpy="${o_rpy}"/>
-            <inertia    ixx="${(1/12) * m * (3*r*r+l*l)}"   ixy="0"   ixz="0"
-                        iyy="${(1/12) * m * (3*r*r+l*l)}"   iyz="0"
-                        izz="${(1/12) *m*r*r}"   />
-        </inertial>
-    </xacro:macro>
-    <xacro:macro name="sphere_collition_inertia" params="m r o_xyz o_rpy">
-        <collision>
-            <geometry>
-                <sphere radius="${wheel_radius / 2.0}" />
-            </geometry>
-            <origin xyz="0 0 0" rpy="0 0 0" />
-        </collision>
-        <inertial>
-            <mass value="${m}"/>
-            <origin xyz="${o_xyz}" rpy="${o_rpy}"/>
-            <inertia    ixx="${(2/5) * m * r*r}"   ixy="0"   ixz="0"
-                        iyy="${(2/5) * m * r*r}"   iyz="0"
-                        izz="${(2/5) * m * r*r}"   />
-        </inertial>
-    </xacro:macro>
-</robot>
+/home/vincent-pc/ros2_jazzy/src/my_robot_description/urdf/common_properties.xacro

File: install/my_robot_description/share/my_robot_description/urdf/mobile_base.xacro (robot description, xacro)
@@ -1,68 +1 @@
-<?xml version="1.0"?>
-<robot xmlns:xacro="http://www.ros.org/wiki/xacro">
-    <xacro:property name="base_length" value="0.6" />
-    <xacro:property name="base_width" value="0.4" />
-    <xacro:property name="base_height" value="0.2" />
-    <xacro:property name="wheel_radius" value="0.1" />
-    <xacro:property name="wheel_length" value="0.05" />
-    <link name="base_footprint" />
-    <link name="base_link">
-        <visual>
-            <geometry>
-                <box size="${base_length} ${base_width} ${base_height}" />
-            </geometry>
-            <origin xyz="0 0 ${base_height / 2.0}" rpy="0 0 0" />
-            <material name="red" />
-        </visual>
-        <xacro:box_collition_inertia m="5.0" x="${base_length}" y="${base_width}" z="${base_height}"
-                           o_xyz="0 0 ${base_height / 2.0}" o_rpy="0 0 0" />
-    </link>
-    <xacro:macro name="wheel_link" params="prefix">
-        <link name="${prefix}_wheel_link">
-            <visual>
-                <geometry>
-                    <cylinder radius="${wheel_radius}" length="${wheel_length}" />
-                </geometry>
-                <origin xyz="0 0 0" rpy="${pi / 2.0} 0 0" />
-                <material name="purple" />
-            </visual>
-            <xacro:cylinder_collition_inertia m="1.0" r="${wheel_radius}" l="${wheel_length}"
-                                    o_xyz="0 0 0" o_rpy="${pi / 2.0} 0 0" />
-        </link>
-    </xacro:macro>
-    <xacro:wheel_link prefix="right" />
-    <xacro:wheel_link prefix="left" />
-    <link name="caster_wheel_link">
-        <visual>
-            <geometry>
-                <sphere radius="${wheel_radius / 2.0}" />
-            </geometry>
-            <origin xyz="0 0 0" rpy="0 0 0" />
-            <material name="purple" />
-        </visual>
-        <xacro:sphere_collition_inertia m="0.5" r="${wheel_radius / 2.0}"
-                              o_xyz="0 0 0" o_rpy="0 0 0" />
-    </link>
-    <joint name="base_joint" type="fixed">
-        <parent link="base_footprint" />
-        <child link="base_link" />
-        <origin xyz="0 0 ${wheel_radius}" rpy="0 0 0"/>
-    </joint>
-    <joint name="base_right_wheel_joint" type="continuous">
-        <parent link="base_link" />
-        <child link="right_wheel_link" />
-        <origin xyz="${-base_length / 4.0} ${-(base_width + wheel_length) / 2.0} 0" rpy="0 0 0" />
-        <axis xyz="0 1 0" />
-    </joint>
-    <joint name="base_left_wheel_joint" type="continuous">
-        <parent link="base_link" />
-        <child link="left_wheel_link" />
-        <origin xyz="${-base_length / 4.0} ${(base_width + wheel_length) / 2.0} 0" rpy="0 0 0" />
-        <axis xyz="0 1 0" />
-    </joint>
-    <joint name="base_caster_wheel_joint" type="fixed">
-        <parent link="base_link" />
-        <child link="caster_wheel_link" />
-        <origin xyz="${base_length / 3.0} 0 ${-wheel_radius / 2.0}" rpy="0 0 0" />
-    </joint>
-</robot>
+/home/vincent-pc/ros2_jazzy/src/my_robot_description/urdf/mobile_base.xacro

File: install/my_robot_description/share/my_robot_description/urdf/mobile_base_Vinc.xacro (robot description, xacro)
@@ -1,70 +1 @@
-<?xml version="1.0"?>
-<robot xmlns:xacro="http://www.ros.org/wiki/xacro" >
-    <xacro:property name="base_length" value="0.6"/>
-    <xacro:property name="base_width" value="0.4"/>
-    <xacro:property name="base_height" value="0.2"/>
-    <xacro:property name="wheel_radius" value="0.1"/>
-    <xacro:property name="wheel_length" value="0.05"/>
-    <xacro:property name="wheel_caster_radius" value="0.05"/>
-    <link name="base_footprint" />
-    <link name="base_link">
-        <visual>
-            <geometry>
-                <box size="${base_length} ${base_width} ${base_height}" />
-            </geometry>
-            <origin xyz="0 0 ${base_height/2.0}" rpy="0 0 0" />
-            <material name="purple" />
-        </visual>
-        <xacro:box_collition_inertia m="5.0" x="${base_length}" y="${base_width}" z="${base_height}"
-                            o_xyz="0 0 ${base_height/2.0}" o_rpy="0 0 0" />
-    </link>
-    <xacro:macro name="wheel_link" params="prefix">
-        <link name="${prefix}_wheel_link">
-            <visual>
-                <geometry>
-                    <cylinder radius="${wheel_radius}" length="${wheel_length}" />
-                </geometry>
-                <origin xyz="0 0 0.0" rpy= "${pi/2.0} 0 0" />
-                <material name="red" />
-            </visual>
-            <xacro:cylinder_collition_inertia m="1.0" r="${wheel_radius}" l="${wheel_length}"
-                            o_xyz="0 0 0" o_rpy="${pi/2.0} 0 0" />
-        </link>
-    </xacro:macro>
-    <xacro:wheel_link prefix="right" />
-    <xacro:wheel_link prefix="left" />
-    <link name="base_caster_wheel_link">
-        <visual>
-            <geometry>
-                <sphere radius="${wheel_caster_radius}" />
-            </geometry>
-            <origin xyz="0 0 0" rpy= "0 0 0" />
-            <material name="red" />
-        </visual>
-        <xacro:sphere_collition_inertia m="1.0" r="${wheel_caster_radius}"
-                            o_xyz="0 0 0" o_rpy="0 0 0" />
-    </link>
-    <joint name="base_footprint_joint" type="fixed">
-        <parent link="base_footprint"/>
-        <child link="base_link"/>
-        <origin xyz="0 0 ${wheel_radius}" rpy="0 0 0"/>
-    </joint>
-    <joint name="base_right_wheel_joint" type="continuous">
-        <parent link="base_link"/>
-        <child link="right_wheel_link"/>
-        <origin xyz="${- base_length/4.0} ${-(base_width+wheel_length)/2.0} 0" rpy="0 0 0"/>
-        <axis xyz="0 1 0"/>
-    </joint>
-    <joint name="base_left_wheel_joint" type="continuous">
-        <parent link="base_link"/>
-        <child link="left_wheel_link"/>
-        <origin xyz="${- base_length/4.0} ${(base_width+wheel_length)/2.0} 0" rpy="0 0 0"/>
-        <axis xyz="0 1 0"/>
-    </joint>
-    <joint name="base_caster_wheel_joint" type="fixed">
-        <parent link="base_link"/>
-        <child link="base_caster_wheel_link"/>
-        <origin xyz="${base_length/3.0} 0 ${-wheel_radius/2.0}" rpy="0 0 0"/>
-        <axis xyz="0 0 0"/>
-    </joint>
-</robot>
+/home/vincent-pc/ros2_jazzy/src/my_robot_description/urdf/mobile_base_Vinc.xacro

File: install/my_robot_description/share/my_robot_description/urdf/mobile_base_gz.xacro (robot description, xacro)
@@ -1,27 +1 @@
-<?xml version="1.0"?>
-<robot xmlns:xacro="http://www.ros.org/wiki/xacro" >
-    <gazebo reference="caster_wheel_link">
-        <mu1 value="0.1" />
-        <mu2 value="0.1" />
-    </gazebo>
-    <gazebo>
-        <plugin
-            filename="gz-sim-diff-drive-system"
-            name="gz::sim::systems::DiffDrive">
-            <left_joint>base_left_wheel_joint</left_joint>
-            <right_joint>base_right_wheel_joint</right_joint>
-            <wheel_separation>0.45</wheel_separation>
-            <wheel_radius>0.1</wheel_radius>
-            <frame_id>odom</frame_id>
-            <child_frame_id>base_footprint</child_frame_id>
-        </plugin>
-    </gazebo>
-    <gazebo>
-        <plugin
-            filename="gz-sim-joint-state-publisher-system"
-            name="gz::sim::systems::JointStatePublisher">
-            <joint_name>base_left_wheel_joint</joint_name>
-            <joint_name>base_right_wheel_joint</joint_name>
-        </plugin>
-    </gazebo>
-</robot>
+/home/vincent-pc/ros2_jazzy/src/my_robot_description/urdf/mobile_base_gz.xacro

File: install/my_robot_description/share/my_robot_description/urdf/my_robot.urdf.xacro (robot description, xacro)
@@ -1,7 +1 @@
-<?xml version="1.0"?>
-<robot name="my_robot" xmlns:xacro="http://www.ros.org/wiki/xacro" >
-    <xacro:include filename="common_properties.xacro" />
-    <xacro:include filename="mobile_base.xacro"/>
-    <!-- <xacro:include filename="mobile_base_Vinc.xacro"/> -->
-    <xacro:include filename="mobile_base_gz.xacro"/>
-</robot>
+/home/vincent-pc/ros2_jazzy/src/my_robot_description/urdf/my_robot.urdf.xacro

File: src/my_robot_description/urdf/common_properties.xacro (robot description, xacro)
@@ -6,4 +6,10 @@
     <material name="red">
         <color rgba="1 0 0 1" />
+    </material>
+    <material name="orange">
+        <color rgba="1.0 0.5 0 1" />
+    </material>
+    <material name="yellow">
+        <color rgba="1.0 1.0 0 1" />
     </material>
     <xacro:macro name="box_collition_inertia" params="m x y z o_xyz o_rpy">
@@ -37,4 +43,19 @@
         </inertial>
     </xacro:macro>
+    <xacro:macro name="cylinder2_collition_inertia" params="m r l o_xyz o_rpy">
+        <collision>
+                <geometry>
+                    <cylinder radius="${r}" length="${l}"/>
+                </geometry>
+                <origin xyz="${o_xyz}" rpy="0 0 0" />
+            </collision>
+        <inertial>
+            <mass value="${m}"/>
+            <origin xyz="${o_xyz}" rpy="${o_rpy}"/>
+            <inertia    ixx="${(1/12) * m * (3*r*r+l*l)}"   ixy="0"   ixz="0"
+                        iyy="${(1/12) * m * (3*r*r+l*l)}"   iyz="0"
+                        izz="${(1/12) *m*r*r}"   />
+        </inertial>
+    </xacro:macro>
     <xacro:macro name="sphere_collition_inertia" params="m r o_xyz o_rpy">
         <collision>

File: src/my_robot_description/urdf/my_robot.urdf.xacro (robot description, xacro)
@@ -5,3 +5,11 @@
     <!-- <xacro:include filename="mobile_base_Vinc.xacro"/> -->
     <xacro:include filename="mobile_base_gz.xacro"/>
+    <xacro:include filename="arm.xacro"/>
+    <xacro:include filename="arm_gazebo.xacro"/>
+    <xacro:include filename="camera.xacro" />
+    <joint name="mobile_base_arm_joint" type="fixed">
+        <parent link="base_link"/>
+        <child link="arm_base_link"/>
+        <origin xyz="${base_length/4} 0.0 ${base_height}" rpy="0.0 0.0 0.0"/>
+    </joint>
 </robot>

File: src/my_robot_description/urdf/test.urdf (robot description, URDF)
Before this commit: robot my_robot, 5 links, 4 joints
Links:
- removed link base_caster_wheel_link
- removed link base_footprint
- removed link base_link
- removed link left_wheel_link
- removed link right_wheel_link
- added link arm_base_link; visual box size=0.1 0.1 0.02
- added link first_arm_link; visual cylinder length=0.3 radius=0.02
Joints:
- removed joint base_caster_wheel_joint
- removed joint base_footprint_joint
- removed joint base_left_wheel_joint
- removed joint base_right_wheel_joint
- added joint first_joint: type revolute, parent arm_base_link, child first_arm_link, origin xyz=0 0 0.16999999999999998 rpy=0 0 0, axis 0 0 0, limit lower=0.0 upper=1.5707963267948966 effort=100 velocity=100
