Commit message: Turtlesim and TurtleBot3 using ROS2 actions, lifecycle and component

File: install/my_robot_description/share/my_robot_description/urdf/arm.xacro (robot description, xacro)
@@ -1 +1,104 @@
-/home/vincent-pc/ros2_jazzy/src/my_robot_description/urdf/arm.xacro
+<?xml version="1.0"?>
+<robot xmlns:xacro="http://www.ros.org/wiki/xacro">
+    <xacro:property name="arm_base_length" value="0.1" />
+    <xacro:property name="arm_base_width" value="0.1" />
+    <xacro:property name="arm_base_height" value="0.02" />
+    <xacro:property name="gripper_base_length" value="0.05" />
+    <xacro:property name="gripper_base_width" value="0.1" />
+    <xacro:property name="gripper_base_height" value="0.02" />
+    <xacro:property name="arm_radius" value="0.02" />
+    <xacro:property name="arm_length" value="0.3" />
+    <xacro:property name="gripper_radius" value="0.015" />
+    <xacro:property name="gripper_length" value="0.1" />
+    <link name="arm_base_link">
+        <visual>
+            <geometry>
+                <box size="${arm_base_length} ${arm_base_width} ${arm_base_height}" />
+            </geometry>
+            <origin xyz="0 0 ${arm_base_height / 2.0}" rpy="0 0 0" />
+            <material name="yellow" />
+        </visual>
+        <xacro:box_collition_inertia m="0.5" x="${arm_base_length}" y="${arm_base_width}" z="${arm_base_height}"
+                           o_xyz="0 0 ${arm_base_height / 2.0}" o_rpy="0 0 0" />
+    </link>
+    <!-- PRIMER BRAZO -->
+    <xacro:macro name="arm_link" params="prefix color o_xyz">
+        <link name="${prefix}_arm_link">
+            <visual>
+                <geometry>
+                    <cylinder radius="${arm_radius}" length="${arm_length}" />
+                </geometry>
+                <origin xyz="${o_xyz}" rpy="0 0 0" />
+                <material name="${color}" />
+            </visual>
+            <xacro:cylinder2_collition_inertia m="0.3" r="${arm_radius}" l="${arm_length}"
+                                    o_xyz="${o_xyz}" o_rpy="0 0 0" />
+        </link>
+    </xacro:macro>
+    <xacro:arm_link prefix="first" color="purple" o_xyz="0 0 ${arm_length/2}" />
+    <xacro:arm_link prefix="hand" color="red" o_xyz="0 0 ${arm_length/2}" />
+    <link name="gripper_base_link">
+        <visual>
+            <geometry>
+                <box size="${gripper_base_length} ${gripper_base_width} ${gripper_base_height}" />
+            </geometry>
+            <origin xyz="0 0 ${gripper_base_height / 2.0}" rpy="0 0 0" />
+            <material name="yellow" />
+        </visual>
+        <xacro:box_collition_inertia m="0.5" x="${gripper_base_length}" y="${gripper_base_width}" z="${gripper_base_height}"
+                           o_xyz="0 0 ${gripper_base_height / 2.0}" o_rpy="0 0 0" />
+    </link>
+    <!-- gripper -->
+    <xacro:macro name="gripper_link" params="prefix color o_xyz">
+        <link name="${prefix}_gripper_link">
+            <visual>
+                <geometry>
+                    <cylinder radius="${gripper_radius}" length="${gripper_length}" />
+                </geometry>
+                <origin xyz="${o_xyz}" rpy="0 0 0" />
+                <material name="${color}" />
+            </visual>
+            <xacro:cylinder2_collition_inertia m="0.3" r="${gripper_radius}" l="${gripper_length}"
+                                    o_xyz="${o_xyz}" o_rpy="0 0 0" />
+        </link>
+    </xacro:macro>
+    <xacro:gripper_link prefix="left" color="purple" o_xyz="0 0 ${gripper_length/2}" />
+    <xacro:gripper_link prefix="right" color="purple" o_xyz="0 0 ${gripper_length/2}" />
+    <joint name="first_joint" type="revolute">
+        <parent link="arm_base_link"/>
+        <child link="first_arm_link"/>
+        <origin xyz="0 0 ${arm_base_height}" rpy="0 0 0"/>
+        <axis xyz="0 1 0"/>
+        <limit lower="0" upper="${pi/2}" effort="100" velocity="100"/>
+        <dynamics friction="0.3" damping="0.3" />
+    </joint>
+    <joint name="second_joint" type="revolute">
+        <parent link="first_arm_link" />
+        <child link="hand_arm_link" />
+        <origin xyz="0 0 ${arm_length}" rpy="0 0 0" />
+        <axis xyz="0 1 0" />
+        <limit lower="0.0" upper="${pi/2}" effort="100" velocity="100"/>
+        <dynamics friction="0.3" damping="0.3" />
+    </joint>
+    <joint name="gripper_base_joint" type="fixed">
+        <parent link="hand_arm_link"/>
+        <child link="gripper_base_link"/>
+        <origin xyz="0.0 0.0 ${arm_length}" rpy="0.0 0.0 0.0"/>
+    </joint>
+    <joint name="gripper_left_joint" type="revolute">
+        <parent link="gripper_base_link"/>
+        <child link="left_gripper_link"/>
+        <origin xyz="0 -0.05 ${gripper_base_height}" rpy="0 0 0"/>
+        <axis xyz="-1 0 0"/>
+        <limit lower="0" upper="${pi/2}" effort="100" velocity="100"/>
+        <dynamics friction="0.3" damping="0.3" />
+    </joint>
+    <joint name="gripper_right_joint" type="revolute">
+        <parent link="gripper_base_link"/>
+        <child link="right_gripper_link"/>
+        <origin xyz="0 0.05 ${gripper_base_height}" rpy="0 0 0"/>
+        <axis xyz="1 0 0"/>
+        <limit lower="0" upper="${pi/2}" effort="100" velocity="100"/>
+        <dynamics friction="0.3" damping="0.3" />
+    </joint>
+</robot>

File: install/my_robot_description/share/my_robot_description/urdf/arm_gazebo.xacro (robot description, xacro)
@@ -1 +1,46 @@
-/home/vincent-pc/ros2_jazzy/src/my_robot_description/urdf/arm_gazebo.xacro
+<?xml version="1.0"?>
+<robot xmlns:xacro="http://www.ros.org/wiki/xacro" >
+    <!-- https://github.com/gazebosim/gz-sim/tree/gz-sim9/src/systems -->
+    <gazebo>
+        <plugin
+            filename="gz-sim-joint-position-controller-system"
+            name="gz::sim::systems::JointPositionController" >
+            <joint_name>first_joint</joint_name>
+            <p_gain>10.0</p_gain>
+        </plugin>
+    </gazebo>
+    <gazebo>
+        <plugin
+            filename="gz-sim-joint-position-controller-system"
+            name="gz::sim::systems::JointPositionController" >
+            <joint_name>second_joint</joint_name>
+            <p_gain>6.0</p_gain>
+        </plugin>
+    </gazebo>
+    <gazebo>
+        <plugin
+            filename="gz-sim-joint-position-controller-system"
+            name="gz::sim::systems::JointPositionController" >
+            <joint_name>gripper_left_joint</joint_name>
+            <p_gain>3.0</p_gain>
+        </plugin>
+    </gazebo>
+    <gazebo>
+        <plugin
+            filename="gz-sim-joint-position-controller-system"
+            name="gz::sim::systems::JointPositionController" >
+            <joint_name>gripper_right_joint</joint_name>
+            <p_gain>3.0</p_gain>
+        </plugin>
+    </gazebo>
+    <gazebo>
+        <plugin
+            filename="gz-sim-joint-state-publisher-system"
+            name="gz::sim::systems::JointStatePublisher">
+            <joint_name>first_joint</joint_name>
+            <joint_name>second_joint</joint_name>
+            <joint_name>gripper_left_joint</joint_name>
+            <joint_name>gripper_right_joint</joint_name>
+        </plugin>
+    </gazebo>
+</robot>

File: install/my_robot_description/share/my_robot_description/urdf/camera.xacro (robot description, xacro)
@@ -1 +1,53 @@
-/home/vincent-pc/ros2_jazzy/src/my_robot_description/urdf/camera.xacro
+<?xml version="1.0"?>
+<robot xmlns:xacro="http://www.ros.org/wiki/xacro" >
+    <xacro:property name="camera_length" value="0.01" />
+    <xacro:property name="camera_width" value="0.1" />
+    <xacro:property name="camera_height" value="0.05" />
+    <link name="camera_link">
+        <visual>
+            <geometry>
+                <box size="${camera_length} ${camera_width} ${camera_height}"/>
+            </geometry>
+            <material name="purple"/>
+        </visual>
+        <xacro:box_collition_inertia m="0.1" x="${camera_length}" y="${camera_width}" z="${camera_height}"
+                           o_xyz="0 0 0" o_rpy="0 0 0" />
+    </link>
+    <joint name="base_camera_joint" type="fixed">
+        <parent link="base_link"/>
+        <child link="camera_link"/>
+        <origin xyz="${base_length/2.0+camera_length/2.0} 0.0 ${base_height/2.0}" rpy="0.0 0.0 0.0"/>
+    </joint>
+    <link name="camera_link_optical" />
+    <joint name="camera_optical_joint" type="fixed">
+        <origin xyz="0.0 0.0 0.0" rpy="${-pi/2} 0.0 ${-pi/2}"/>
+        <parent link="camera_link"/>
+        <child link="camera_link_optical"/>
+    </joint>
+    <gazebo reference="camera_link" >
+        <sensor name="camera" type="camera">
+            <camera>
+                <horizontal_fov>1.3962634</horizontal_fov>
+                <image>
+                    <width>640</width>
+                    <height>480</height>
+                    <format>R8G8B8</format>
+                </image>
+                <clip>
+                    <near>0.1</near>
+                    <far>15</far>
+                </clip>
+                <noise>
+                    <type>gaussian</type>
+                    <mean>0.0</mean>
+                    <stddev>0.007</stddev>
+                </noise>
+                <optical_frame_id>camera_link_optical</optical_frame_id>
+                <camera_info_topic>camera/camera_info</camera_info_topic>
+            </camera>
+            <always_on>1</always_on>
+            <update_rate>20</update_rate>
+            <topic>camera/image_raw</topic>
+        </sensor>
+    </gazebo>
+</robot>

File: install/my_robot_description/share/my_robot_description/urdf/common_properties.xacro (robot description, xacro)
@@ -1 +1,75 @@
-/home/vincent-pc/ros2_jazzy/src/my_robot_description/urdf/common_properties.xacro
+<?xml version="1.0"?>
+<robot xmlns:xacro="http://www.ros.org/wiki/xacro" >
+    <material name="purple">
+        <color rgba="0.5 0 0.5 1" />
+    </material>
+    <material name="red">
+        <color rgba="1 0 0 1" />
+    </material>
+    <material name="orange">
+        <color rgba="1.0 0.5 0 1" />
+    </material>
+    <material name="yellow">
+        <color rgba="1.0 1.0 0 1" />
+    </material>
+    <xacro:macro name="box_collition_inertia" params="m x y z o_xyz o_rpy">
+        <collision>
+            <geometry>
+                <box size="${x} ${y} ${z}" />
+            </geometry>
+            <origin xyz="0 0 ${z / 2.0}" rpy="0 0 0" />
+        </collision>
+        <inertial>
+            <mass value="${m}"/>
+            <origin xyz="${o_xyz}" rpy="${o_rpy}"/>
+            <inertia    ixx="${(m/12) * (y*y + z*z)}"   ixy="0"   ixz="0"
+                        iyy="${(m/12) * (x*x + z*z)}"   iyz="0"
+                        izz="${(m/12) * (x*x + y*y)}"   />
+        </inertial>
+    </xacro:macro>
+    <xacro:macro name="cylinder_collition_inertia" params="m r l o_xyz o_rpy">
+        <collision>
+                <geometry>
+                    <sphere radius="${r}" />
+                </geometry>
+                <origin xyz="0 0 0" rpy="0 0 0" />
+            </collision>
+        <inertial>
+            <mass value="${m}"/>
+            <origin xyz="${o_xyz}" rpy="${o_rpy}"/>
+            <inertia    ixx="${(1/12) * m * (3*r*r+l*l)}"   ixy="0"   ixz="0"
+                        iyy="${(1/12) * m * (3*r*r+l*l)}"   iyz="0"
+                        izz="${(1/12) *m*r*r}"   />
+        </inertial>
+    </xacro:macro>
+    <xacro:macro name="cylinder2_collition_inertia" params="m r l o_xyz o_rpy">
+        <collision>
+                <geometry>
+                    <cylinder radius="${r}" length="${l}"/>
+                </geometry>
+                <origin xyz="${o_xyz}" rpy="0 0 0" />
+            </collision>
+        <inertial>
+            <mass value="${m}"/>
+            <origin xyz="${o_xyz}" rpy="${o_rpy}"/>
+            <inertia    ixx="${(1/12) * m * (3*r*r+l*l)}"   ixy="0"   ixz="0"
+                        iyy="${(1/12) * m * (3*r*r+l*l)}"   iyz="0"
+                        izz="${(1/12) *m*r*r}"   />
+        </inertial>
+    </xacro:macro>
+    <xacro:macro name="sphere_collition_inertia" params="m r o_xyz o_rpy">
+        <collision>
+            <geometry>
+                <sphere radius="${wheel_radius / 2.0}" />
+            </geometry>
+            <origin xyz="0 0 0" rpy="0 0 0" />
+        </collision>
+        <inertial>
+            <mass value="${m}"/>
+            <origin xyz="${o_xyz}" rpy="${o_rpy}"/>
+            <inertia    ixx="${(2/5) * m * r*r}"   ixy="0"   ixz="0"
+                        iyy="${(2/5) * m * r*r}"   iyz="0"
+                        izz="${(2/5) * m * r*r}"   />
+        </inertial>
+    </xacro:macro>
+</robot>

File: install/my_robot_description/share/my_robot_description/urdf/mobile_base.xacro (robot description, xacro)
@@ -1 +1,68 @@
-/home/vincent-pc/ros2_jazzy/src/my_robot_description/urdf/mobile_base.xacro
+<?xml version="1.0"?>
+<robot xmlns:xacro="http://www.ros.org/wiki/xacro">
+    <xacro:property name="base_length" value="0.6" />
+    <xacro:property name="base_width" value="0.4" />
+    <xacro:property name="base_height" value="0.2" />
+    <xacro:property name="wheel_radius" value="0.1" />
+    <xacro:property name="wheel_length" value="0.05" />
+    <link name="base_footprint" />
+    <link name="base_link">
+        <visual>
+            <geometry>
+                <box size="${base_length} ${base_width} ${base_height}" />
+            </geometry>
+            <origin xyz="0 0 ${base_height / 2.0}" rpy="0 0 0" />
+            <material name="red" />
+        </visual>
+        <xacro:box_collition_inertia m="5.0" x="${base_length}" y="${base_width}" z="${base_height}"
+                           o_xyz="0 0 ${base_height / 2.0}" o_rpy="0 0 0" />
+    </link>
+    <xacro:macro name="wheel_link" params="prefix">
+        <link name="${prefix}_wheel_link">
+            <visual>
+                <geometry>
+                    <cylinder radius="${wheel_radius}" length="${wheel_length}" />
+                </geometry>
+                <origin xyz="0 0 0" rpy="${pi / 2.0} 0 0" />
+                <material name="purple" />
+            </visual>
+            <xacro:cylinder_collition_inertia m="1.0" r="${wheel_radius}" l="${wheel_length}"
+                                    o_xyz="0 0 0" o_rpy="${pi / 2.0} 0 0" />
+        </link>
+    </xacro:macro>
+    <xacro:wheel_link prefix="right" />
+    <xacro:wheel_link prefix="left" />
+    <link name="caster_wheel_link">
+        <visual>
+            <geometry>
+                <sphere radius="${wheel_radius / 2.0}" />
+            </geometry>
+            <origin xyz="0 0 0" rpy="0 0 0" />
+            <material name="purple" />
+        </visual>
+        <xacro:sphere_collition_inertia m="0.5" r="${wheel_radius / 2.0}"
+                              o_xyz="0 0 0" o_rpy="0 0 0" />
+    </link>
+    <joint name="base_joint" type="fixed">
+        <parent link="base_footprint" />
+        <child link="base_link" />
+        <origin xyz="0 0 ${wheel_radius}" rpy="0 0 0"/>
+    </joint>
+    <joint name="base_right_wheel_joint" type="continuous">
+        <parent link="base_link" />
+        <child link="right_wheel_link" />
+        <origin xyz="${-base_length / 4.0} ${-(base_width + wheel_length) / 2.0} 0" rpy="0 0 0" />
+        <axis xyz="0 1 0" />
+    </joint>
+    <joint name="base_left_wheel_joint" type="continuous">
+        <parent link="base_link" />
+        <child link="left_wheel_link" />
+        <origin xyz="${-base_length / 4.0} ${(base_width + wheel_length) / 2.0} 0" rpy="0 0 0" />
+        <axis xyz="0 1 0" />
+    </joint>
+    <joint name="base_caster_wheel_joint" type="fixed">
+        <parent link="base_link" />
+        <child link="caster_wheel_link" />
+        <origin xyz="${base_length / 3.0} 0 ${-wheel_radius / 2.0}" rpy="0 0 0" />
+    </joint>
+</robot>

File: install/my_robot_description/share/my_robot_description/urdf/mobile_base_Vinc.xacro (robot description, xacro)
@@ -1 +1,70 @@
-/home/vincent-pc/ros2_jazzy/src/my_robot_description/urdf/mobile_base_Vinc.xacro
+<?xml version="1.0"?>
+<robot xmlns:xacro="http://www.ros.org/wiki/xacro" >
+    <xacro:property name="base_length" value="0.6"/>
+    <xacro:property name="base_width" value="0.4"/>
+    <xacro:property name="base_height" value="0.2"/>
+    <xacro:property name="wheel_radius" value="0.1"/>
+    <xacro:property name="wheel_length" value="0.05"/>
+    <xacro:property name="wheel_caster_radius" value="0.05"/>
+    <link name="base_footprint" />
+    <link name="base_link">
+        <visual>
+            <geometry>
+                <box size="${base_length} ${base_width} ${base_height}" />
+            </geometry>
+            <origin xyz="0 0 ${base_height/2.0}" rpy="0 0 0" />
+            <material name="purple" />
+        </visual>
+        <xacro:box_collition_inertia m="5.0" x="${base_length}" y="${base_width}" z="${base_height}"
+                            o_xyz="0 0 ${base_height/2.0}" o_rpy="0 0 0" />
+    </link>
+    <xacro:macro name="wheel_link" params="prefix">
+        <link name="${prefix}_wheel_link">
+            <visual>
+                <geometry>
+                    <cylinder radius="${wheel_radius}" length="${wheel_length}" />
+                </geometry>
+                <origin xyz="0 0 0.0" rpy= "${pi/2.0} 0 0" />
+                <material name="red" />
+            </visual>
+            <xacro:cylinder_collition_inertia m="1.0" r="${wheel_radius}" l="${wheel_length}"
+                            o_xyz="0 0 0" o_rpy="${pi/2.0} 0 0" />
+        </link>
+    </xacro:macro>
+    <xacro:wheel_link prefix="right" />
+    <xacro:wheel_link prefix="left" />
+    <link name="base_caster_wheel_link">
+        <visual>
+            <geometry>
+                <sphere radius="${wheel_caster_radius}" />
+            </geometry>
+            <origin xyz="0 0 0" rpy= "0 0 0" />
+            <material name="red" />
+        </visual>
+        <xacro:sphere_collition_inertia m="1.0" r="${wheel_caster_radius}"
+                            o_xyz="0 0 0" o_rpy="0 0 0" />
+    </link>
+    <joint name="base_footprint_joint" type="fixed">
+        <parent link="base_footprint"/>
+        <child link="base_link"/>
+        <origin xyz="0 0 ${wheel_radius}" rpy="0 0 0"/>
+    </joint>
+    <joint name="base_right_wheel_joint" type="continuous">
+        <parent link="base_link"/>
+        <child link="right_wheel_link"/>
+        <origin xyz="${- base_length/4.0} ${-(base_width+wheel_length)/2.0} 0" rpy="0 0 0"/>
+        <axis xyz="0 1 0"/>
+    </joint>
+    <joint name="base_left_wheel_joint" type="continuous">
+        <parent link="base_link"/>
+        <child link="left_wheel_link"/>
+        <origin xyz="${- base_length/4.0} ${(base_width+wheel_length)/2.0} 0" rpy="0 0 0"/>
+        <axis xyz="0 1 0"/>
+    </joint>
+    <joint name="base_caster_wheel_joint" type="fixed">
+        <parent link="base_link"/>
+        <child link="base_caster_wheel_link"/>
+        <origin xyz="${base_length/3.0} 0 ${-wheel_radius/2.0}" rpy="0 0 0"/>
+        <axis xyz="0 0 0"/>
+    </joint>
+</robot>

File: install/my_robot_description/share/my_robot_description/urdf/mobile_base_gz.xacro (robot description, xacro)
@@ -1 +1,27 @@
-/home/vincent-pc/ros2_jazzy/src/my_robot_description/urdf/mobile_base_gz.xacro
+<?xml version="1.0"?>
+<robot xmlns:xacro="http://www.ros.org/wiki/xacro" >
+    <gazebo reference="caster_wheel_link">
+        <mu1 value="0.1" />
+        <mu2 value="0.1" />
+    </gazebo>
+    <gazebo>
+        <plugin
+            filename="gz-sim-diff-drive-system"
+            name="gz::sim::systems::DiffDrive">
+            <left_joint>base_left_wheel_joint</left_joint>
+            <right_joint>base_right_wheel_joint</right_joint>
+            <wheel_separation>0.45</wheel_separation>
+            <wheel_radius>0.1</wheel_radius>
+            <frame_id>odom</frame_id>
+            <child_frame_id>base_footprint</child_frame_id>
+        </plugin>
+    </gazebo>
+    <gazebo>
+        <plugin
+            filename="gz-sim-joint-state-publisher-system"
+            name="gz::sim::systems::JointStatePublisher">
+            <joint_name>base_left_wheel_joint</joint_name>
+            <joint_name>base_right_wheel_joint</joint_name>
+        </plugin>
+    </gazebo>
+</robot>

File: install/my_robot_description/share/my_robot_description/urdf/my_arm.urdf.xacro (robot description, xacro)
@@ -1 +1,8 @@
-/home/vincent-pc/ros2_jazzy/src/my_robot_description/urdf/my_arm.urdf.xacro
+<?xml version="1.0"?>
+<robot name="my_robot" xmlns:xacro="http://www.ros.org/wiki/xacro" >
+    <xacro:include filename="common_properties.xacro" />
+    <xacro:include filename="arm.xacro"/>
+    <xacro:include filename="arm_gazebo.xacro"/>
+    <!-- <xacro:include filename="mobile_base_gz.xacro"/>
+    <xacro:include filename="camera.xacro" /> -->
+</robot>

File: install/my_robot_description/share/my_robot_description/urdf/my_robot.urdf.xacro (robot description, xacro)
@@ -1 +1,15 @@
-/home/vincent-pc/ros2_jazzy/src/my_robot_description/urdf/my_robot.urdf.xacro
+<?xml version="1.0"?>
+<robot name="my_robot" xmlns:xacro="http://www.ros.org/wiki/xacro" >
+    <xacro:include filename="common_properties.xacro" />
+    <xacro:include filename="mobile_base.xacro"/>
+    <!-- <xacro:include filename="mobile_base_Vinc.xacro"/> -->
+    <xacro:include filename="mobile_base_gz.xacro"/>
+    <xacro:include filename="arm.xacro"/>
+    <xacro:include filename="arm_gazebo.xacro"/>
+    <xacro:include filename="camera.xacro" />
+    <joint name="mobile_base_arm_joint" type="fixed">
+        <parent link="base_link"/>
+        <child link="arm_base_link"/>
+        <origin xyz="${base_length/4} 0.0 ${base_height}" rpy="0.0 0.0 0.0"/>
+    </joint>
+</robot>
