Commit message: Update code and ros2_control

File: install/my_robot_description/share/my_robot_description/urdf/mobile_base.xacro (robot description, xacro)
@@ -24,9 +24,9 @@
                     <cylinder radius="${wheel_radius}" length="${wheel_length}" />
                 </geometry>
-                <origin xyz="0 0 0" rpy="${pi / 2.0} 0 0" />
+                <origin xyz="0 0 0" rpy= "${pi/2.0} 0 0" />
                 <material name="purple" />
             </visual>
             <xacro:cylinder_collition_inertia m="1.0" r="${wheel_radius}" l="${wheel_length}"
-                                    o_xyz="0 0 0" o_rpy="${pi / 2.0} 0 0" />
+                            o_xyz="0 0 0" o_rpy="${pi/2.0} 0 0" />
         </link>
     </xacro:macro>
@@ -50,14 +50,14 @@
     </joint>
     <joint name="base_right_wheel_joint" type="continuous">
-        <parent link="base_link" />
-        <child link="right_wheel_link" />
-        <origin xyz="${-base_length / 4.0} ${-(base_width + wheel_length) / 2.0} 0" rpy="0 0 0" />
-        <axis xyz="0 1 0" />
+        <parent link="base_link"/>
+        <child link="right_wheel_link"/>
+        <origin xyz="${- base_length/4.0} ${-(base_width+wheel_length)/2.0} 0" rpy="0 0 0"/>
+        <axis xyz="0 1 0"/>
     </joint>
     <joint name="base_left_wheel_joint" type="continuous">
-        <parent link="base_link" />
-        <child link="left_wheel_link" />
-        <origin xyz="${-base_length / 4.0} ${(base_width + wheel_length) / 2.0} 0" rpy="0 0 0" />
-        <axis xyz="0 1 0" />
+        <parent link="base_link"/>
+        <child link="left_wheel_link"/>
+        <origin xyz="${- base_length/4.0} ${(base_width+wheel_length)/2.0} 0" rpy="0 0 0"/>
+        <axis xyz="0 1 0"/>
     </joint>
     <joint name="base_caster_wheel_joint" type="fixed">

File: install/my_robot_description/share/my_robot_description/urdf/mobile_base_Vinc.xacro (robot description, xacro)
@@ -25,5 +25,5 @@
                     <cylinder radius="${wheel_radius}" length="${wheel_length}" />
                 </geometry>
-                <origin xyz="0 0 0.0" rpy= "${pi/2.0} 0 0" />
+                <origin xyz="0 0 0" rpy= "${pi/2.0} 0 0" />
                 <material name="red" />
             </visual>

File: install/my_robot_description/share/my_robot_description/urdf/my_robot.urdf.xacro (robot description, xacro)
@@ -3,6 +3,6 @@
     <xacro:include filename="common_properties.xacro" />
     <xacro:include filename="mobile_base.xacro"/>
-    <!-- <xacro:include filename="mobile_base_Vinc.xacro"/> -->
     <xacro:include filename="mobile_base_gz.xacro"/>
+    <xacro:include filename="mobile_base.ros2_control.xacro" />
     <xacro:include filename="arm.xacro"/>
     <xacro:include filename="arm_gazebo.xacro"/>
