Commit message: Update of ros2_control practice

File: install/my_robot_description/share/my_robot_description/urdf/mobile_base.ros2_control.xacro (robot description, xacro)
@@ -1,3 +1,19 @@
 <?xml version="1.0"?>
 <robot name="my_robot" xmlns:xacro="http://www.ros.org/wiki/xacro" >
+    <ros2_control name="MobileBaseHardwareInterface" type="system" >
+        <hardware>
+            <plugin>mock_components/GenericSystem</plugin>
+            <param name="calculate_dynamics">true</param>
+        </hardware>
+        <joint name="base_right_wheel_joint">
+            <command_interface name="velocity" />
+            <state_interface name="position" />
+            <state_interface name="velocity" />
+        </joint>
+        <joint name="base_left_wheel_joint">
+            <command_interface name="velocity" />
+            <state_interface name="position" />
+            <state_interface name="velocity" />
+        </joint>
+    </ros2_control>
 </robot>

File: install/my_robot_description/share/my_robot_description/urdf/my_robot.urdf.xacro (robot description, xacro)
@@ -5,5 +5,5 @@
     <xacro:include filename="mobile_base_gz.xacro"/>
     <xacro:include filename="mobile_base.ros2_control.xacro" />
-    <xacro:include filename="arm.xacro"/>
+    <!-- <xacro:include filename="arm.xacro"/>
     <xacro:include filename="arm_gazebo.xacro"/>
     <xacro:include filename="camera.xacro" />
@@ -12,4 +12,4 @@
         <child link="arm_base_link"/>
         <origin xyz="${base_length/4} 0.0 ${base_height}" rpy="0.0 0.0 0.0"/>
-    </joint>
+    </joint> -->
 </robot>

File: src/my_robot_description/urdf/mobile_base.ros2_control.xacro (robot description, xacro)
@@ -7,10 +7,10 @@
         </hardware>
         <joint name="base_right_wheel_joint">
-            <comand_interface name="velocity" />
+            <command_interface name="velocity" />
             <state_interface name="position" />
             <state_interface name="velocity" />
         </joint>
         <joint name="base_left_wheel_joint">
-            <comand_interface name="velocity" />
+            <command_interface name="velocity" />
             <state_interface name="position" />
             <state_interface name="velocity" />
