Commit message: New projects

File: src/my_robot_description/urdf/arm_gazebo.xacro (robot description, xacro)
@@ -7,5 +7,5 @@
             name="gz::sim::systems::JointPositionController" >
             <joint_name>first_joint</joint_name>
-            <p_gain>5.0</p_gain>
+            <p_gain>10.0</p_gain>
         </plugin>
     </gazebo>
@@ -15,5 +15,5 @@
             name="gz::sim::systems::JointPositionController" >
             <joint_name>second_joint</joint_name>
-            <p_gain>3.0</p_gain>
+            <p_gain>6.0</p_gain>
         </plugin>
     </gazebo>

File: src/my_robot_description/urdf/my_robot.urdf (robot description, URDF)
Before this commit: robot my_robot, 5 links, 4 joints
Links:
- removed link base_caster_wheel_link
- removed link base_foodprint
- added link arm_base_link, mass 0.5; collision box size=0.1 0.1 0.02; visual box size=0.1 0.1 0.02
- added link base_footprint
- added link camera_link, mass 0.1; collision box size=0.01 0.1 0.05; visual box size=0.01 0.1 0.05
- added link camera_link_optical
- added link caster_wheel_link, mass 0.5; collision sphere radius=0.05; visual sphere radius=0.05
- added link first_arm_link, mass 0.3; collision cylinder length=0.3 radius=0.02; visual cylinder length=0.3 radius=0.02
- added link gripper_base_link, mass 0.5; collision box size=0.05 0.1 0.02; visual box size=0.05 0.1 0.02
- added link hand_arm_link, mass 0.3; collision cylinder length=0.3 radius=0.02; visual cylinder length=0.3 radius=0.02
- added link left_gripper_link, mass 0.3; collision cylinder length=0.1 radius=0.015; visual cylinder length=0.1 radius=0.015
- added link right_gripper_link, mass 0.3; collision cylinder length=0.1 radius=0.015; visual cylinder length=0.1 radius=0.015
- link base_link: geometry collision box size=0.6 0.4 0.2; visual box size=0.6 0.4 0.2
- link left_wheel_link: mass None -> 1.0; geometry collision sphere radius=0.1; visual cylinder length=0.05 radius=0.1
- link right_wheel_link: mass None -> 1.0; geometry collision sphere radius=0.1; visual cylinder length=0.05 radius=0.1
Joints:
- removed joint base_foodprint_joint
- removed joint base_rigth_wheel_joint
- added joint base_camera_joint: type fixed, parent base_link, child camera_link, origin xyz=0.305 0.0 0.1 rpy=0.0 0.0 0.0
- added joint base_joint: type fixed, parent base_footprint, child base_link, origin xyz=0 0 0.1 rpy=0 0 0
- added joint base_right_wheel_joint: type continuous, parent base_link, child right_wheel_link, origin xyz=-0.15 -0.225 0 rpy=0 0 0, axis 0 1 0
- added joint camera_optical_joint: type fixed, parent camera_link, child camera_link_optical, origin xyz=0.0 0.0 0.0 rpy=-1.5707963267948966 0.0 -1.5707963267948966
- added joint first_joint: type revolute, parent arm_base_link, child first_arm_link, origin xyz=0 0 0.02 rpy=0 0 0, axis 0 1 0, limit lower=0 upper=1.5707963267948966 effort=100 velocity=100
- added joint gripper_base_joint: type fixed, parent hand_arm_link, child gripper_base_link, origin xyz=0.0 0.0 0.3 rpy=0.0 0.0 0.0
- added joint gripper_left_joint: type revolute, parent gripper_base_link, child left_gripper_link, origin xyz=0 -0.05 0.02 rpy=0 0 0, axis -1 0 0, limit lower=0 upper=1.5707963267948966 effort=100 velocity=100
- added joint gripper_right_joint: type revolute, parent gripper_base_link, child right_gripper_link, origin xyz=0 0.05 0.02 rpy=0 0 0, axis 1 0 0, limit lower=0 upper=1.5707963267948966 effort=100 velocity=100
- added joint mobile_base_arm_joint: type fixed, parent base_link, child arm_base_link, origin xyz=0.15 0.0 0.2 rpy=0.0 0.0 0.0
- added joint second_joint: type revolute, parent first_arm_link, child hand_arm_link, origin xyz=0 0 0.3 rpy=0 0 0, axis 0 1 0, limit lower=0.0 upper=1.5707963267948966 effort=100 velocity=100
- joint base_caster_wheel_joint: axis 0 0 0 -> (none); child base_caster_wheel_link -> caster_wheel_link
